File: KICAD/MySensorsPiGw.sch (KiCad schematic (older format))
At the start: 12 parts, among them J1 ANT, J2 CONN_02X20, J3 CONN_01X01, U1 RFM69HW, U2 NRF24L01

Commit message: v2kicad
Parts:
- added C1, C3: 10u, Capacitors_SMD:C_0805, symbol C_Small
- added C2, C4: 100n, Capacitors_SMD:C_0805, symbol C_Small
- added U3: AP1117, TO_SOT_Packages_SMD:SOT-223, symbol AP1117
Connections:
- net +3V3: now also C3.1, C4.1, U3.2 (VO), U3.4 (VO); no longer J2.17 (P17)
- net GND: now also C1.2, C2.2, C3.2, C4.2, U3.1 (GND/ADJ)
- net +5V: now reaches J2.2 (P2)
- net +5V: now also J2.4 (P4), C1.1, C2.1, U3.3 (VI)
Other:
- moved on the sheet: D1, D2, D3, J1, J2, J3, R1, R2, R3, R4, U1, U2

Commit message: v3 kicad
Parts:
- added C5: 10u, Capacitors_SMD:C_0805, symbol C_Small
- added C6: 100n, Capacitors_SMD:C_0805, symbol C_Small
- added D4: ERR, LEDs:LED_0805_HandSoldering, symbol LED
- added D5: RX, LEDs:LED_0805_HandSoldering, symbol LED
- added D6: TX, LEDs:LED_0805_HandSoldering, symbol LED
- added R4, R5, R6: 470, Resistors_SMD:R_0805_HandSoldering, symbol R
- added U4: NRF24L01 SPI1, mysensors_radios:NRF24L01, symbol NRF24L01
- R1, R2, R3: value 1k -> 470
- U2: value NRF24L01 -> NRF24L01 SPI0
- renumbered R4 to R7
Connections:
- net +3V3: now also C5.1, C6.1, R4.1, R5.1, R6.1, U4.2 (VCC)
- net GND: now also C5.2, C6.2, U4.1 (GND)
- net L_ERR_1: now reaches J2.29 (P29)
- net L_ERR_1: now also D4.1 (K)
- net L_RX_1: now reaches J2.31 (P31)
- net L_RX_1: now also D5.1 (K)
- net L_TX_1: now reaches J2.32 (P32)
- net L_TX_1: now also D6.1 (K)
- net IRQ_1: now reaches J2.33 (P33)
- net IRQ_1: now also U4.8 (IRQ)
- net MISO_1: now reaches J2.35 (P35)
- net MISO_1: now also U4.7 (MISO)
- net CS0_1: now reaches J2.36 (P36)
- net CS0_1: now also U4.4 (CSN)
- net CE_1: now reaches J2.37 (P37)
- net CE_1: now also U4.3 (CE)
- net MOSI_1: now reaches J2.38 (P38)
- net MOSI_1: now also U4.6 (MOSI)
- net SCLK_1: now reaches J2.40 (P40)
- net SCLK_1: now also U4.5 (SCK)
- new net: D4.2 (A), R4.2
- new net: D5.2 (A), R5.2
- new net: D6.2 (A), R6.2
Other:
- note added: "Optional NRF24L01 on SPI1"
- note added: "Power"
- note added: "RFM69HW or NRF24L01 on SPI0"
- note added: "Raspberry Pi"
- moved on the sheet: C1, C2, C3, C4, D1, D2, D3, J2, J3, R1, R2, R3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
