File: KICAD/MySensorsPiGw.kicad_pcb (KiCad board)
At the start: 2 copper layers, 65 x 30 mm, 16 parts, among them J1 ANT, J2 CONN_02X20, J3 CONN_01X01, U1 RFM69HW, U2 NRF24L01

Commit message: v2kicad
Parts:
- added C1: 10u, Capacitors_SMD:C_0805, F.Cu at (131.4, 108.6)
- added C2: 100n, Capacitors_SMD:C_0805, F.Cu at (127.8, 108.6)
- added C3: 10u, Capacitors_SMD:C_0805, F.Cu at (131.4, 117.4)
- added C4: 100n, Capacitors_SMD:C_0805, F.Cu at (127.8, 117.4)
- added U3: AP1117, TO_SOT_Packages_SMD:SOT-223, F.Cu at (130.0, 113.0)
- moved R4 1.60 mm to (128.0, 127.0)
Connections:
- J2 pad 17: +3V3 -> Net-(J2-Pad17)
- J2 pad 2: Net-(J2-Pad2) -> +5V
- J2 pad 4: Net-(J2-Pad4) -> +5V
Routing:
- net +5V: track 0.00 -> 14.5 mm
- net GND: track 33.1 -> 40.1 mm, vias 1 -> 7
- net Net-(J3-Pad1): track 2.58 -> 4.29 mm
- net +3V3: track 63.6 -> 63.1 mm, vias 4 -> 3
- net (no net): track 1.21 -> 1.30 mm, vias 42 -> 1
Other:
- net class ant added: clearance 0.2, trace_width 2.4, via_dia 0.6, via_drill 0.4
- board text added: "v2"

Commit message: updatev2
Routing:
- net (no net): track 1.30 -> 0.00 mm, vias 1 -> 0
- net GND: track 40.1 -> 41.4 mm, vias 7 -> 8
Changed lines of the file:
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@@
     (links 51)
     (no_connects 1)
-    (area 115.924999 101.424999 181.075001 131.575001)
+    (area 115.751099 101.253599 181.251101 131.875)
     (thickness 1.6)
     (drawings 62)
-    (tracks 262)
+    (tracks 263)
     (zones 0)
     (modules 21)
@@
   (gr_line (start 116 124) (end 116 128) (angle 90) (layer Edge.Cuts) (width 0.15))
   (gr_line (start 116 105) (end 116 109) (angle 90) (layer Edge.Cuts) (width 0.15))
-  (segment (start 132.4 117.4) (end 133.7 117.4) (width 0.25) (layer B.Cu) (net 0))
-  (via (at 133.7 117.4) (size 0.6) (drill 0.4) (layers F.Cu B.Cu) (net 0))
   (segment (start 156.65 130) (end 155.3 130) (width 0.25) (layer F.Cu) (net 1))
   (segment (start 156.2 106.7) (end 156.1 106.7) (width 0.25) (layer F.Cu) (net 1))
@@
   (segment (start 145.9 102.5) (end 155.6 102.5) (width 0.25) (layer B.Cu) (net 5))
   (segment (start 173.35 126) (end 173.35 130) (width 0.25) (layer F.Cu) (net 6))
-  (segment (start 143.476 122.476) (end 143.424 122.476) (width 0.25) (layer B.Cu) (net 7) (status C00000))
-  (segment (start 143.424 122.476) (end 140.9 125) (width 0.25) (layer B.Cu) (net 7) (status 400000))
+  (segment (start 132.4 117.4) (end 133.552 117.4) (width 0.25) (layer F.Cu) (net 7) (status 400000))
+  (via (at 133.604 117.348) (size 0.6) (drill 0.4) (layers F.Cu B.Cu) (net 7))
+  (segment (start 133.552 117.4) (end 133.604 117.348) (width 0.25) (layer F.Cu) (net 7))
+  (segment (start 143.476 122.476) (end 143.424 122.476) (width 0.25) (layer B.Cu) (net 7))
+  (segment (start 143.424 122.476) (end 140.9 125) (width 0.25) (layer B.Cu) (net 7))
   (segment (start 140.9 125) (end 140.9 126) (width 0.25) (layer B.Cu) (net 7))
   (via (at 140.9 126) (size 0.6) (drill 0.4) (layers F.Cu B.Cu) (net 7))

Commit message: v3 kicad
Parts:
- removed the G*** at (158.1, 118.1)
- added C5: 10u, Capacitors_SMD:C_0805, F.Cu at (159.5, 109.6)
- added C6: 100n, Capacitors_SMD:C_0805, F.Cu at (161.4, 109.6)
- added D4: ERR, LEDs:LED_0805_HandSoldering, F.Cu at (158.0, 126.3)
- added D5: RX, LEDs:LED_0805_HandSoldering, F.Cu at (165.0, 126.2)
- added D6: TX, LEDs:LED_0805_HandSoldering, F.Cu at (172.0, 126.2)
- added R4: 470, Resistors_SMD:R_0805_HandSoldering, F.Cu at (158.0, 124.5)
- added R5: 470, Resistors_SMD:R_0805_HandSoldering, F.Cu at (165.0, 124.4)
- added R6: 470, Resistors_SMD:R_0805_HandSoldering, F.Cu at (170.6, 122.9)
- added U4: NRF24L01 SPI1, mysensors_radios:NRF24L01, F.Cu at (152.1, 108.8)
- R1, R2, R3: value 1k -> 470
- U2: value NRF24L01 -> NRF24L01 SPI0
- moved REF*** 30.6 mm to (136.2, 112.1)
- moved G*** 6.85 mm to (164.6, 114.1)
- moved R1 2.15 mm to (158.0, 128.2)
- moved R2 2.10 mm to (165.0, 128.1)
- moved R3 2.10 mm to (172.0, 128.1)
- moved J3 1.98 mm to (124.0, 127.0)
- renumbered R4 to R7
Connections:
- J2 pad 29: Net-(J2-Pad29) -> /L_ERR_1
- J2 pad 31: Net-(J2-Pad31) -> /L_RX_1
- J2 pad 32: Net-(J2-Pad32) -> /L_TX_1
- J2 pad 33: Net-(J2-Pad33) -> /IRQ_1
- J2 pad 35: Net-(J2-Pad35) -> /MISO_1
- J2 pad 36: Net-(J2-Pad36) -> /CS0_1
- J2 pad 37: Net-(J2-Pad37) -> /CE_1
- J2 pad 38: Net-(J2-Pad38) -> /MOSI_1
- J2 pad 40: Net-(J2-Pad40) -> /SCLK_1
Routing:
- net +3V3: track 63.1 -> 99.2 mm, vias 3 -> 7
- net /L_ERR_1: track 0.00 -> 33.4 mm, vias 0 -> 3
- net /L_TX_1: track 0.00 -> 28.4 mm, vias 0 -> 1
- net /SCLK_1: track 0.00 -> 27.6 mm
- net /MOSI_1: track 0.00 -> 25.4 mm, vias 0 -> 1
- net /L_RX_1: track 0.00 -> 23.8 mm, vias 0 -> 1
- net /MISO_1: track 0.00 -> 23.6 mm, vias 0 -> 1
- net /CS0_1: track 0.00 -> 22.0 mm, vias 0 -> 1
- net /IRQ_1: track 0.00 -> 21.4 mm, vias 0 -> 1
- net /CE_1: track 0.00 -> 21.0 mm
- net GND: track 41.4 -> 52.8 mm, vias 8 -> 9
- net /L_RX: track 54.1 -> 61.1 mm
- net /L_TX: track 54.4 -> 61.4 mm
- net Net-(D6-Pad2): track 0.00 -> 4.21 mm
- net Net-(D1-Pad2): track 4.00 -> 1.85 mm
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Other:
- outline, holes or cut-outs redrawn
- board text added: "RFMHW69"
- board text added: "v3"
- board text removed: "RFMHW69 NRF24L01"
- board text removed: "v2"

Commit message: Add files via upload
Routing:
- net +3V3: track 99.2 -> 104.0 mm, vias 7 -> 8
- net /L_RX_1: track 23.8 -> 24.5 mm
Other:
- net class power added: clearance 0.2, trace_width 0.5, via_dia 0.6, via_drill 0.4
